Commit message: fix: fix something

File: resources/robots/cyberdog2/urdf/cyberdog2.urdf (robot description, URDF)
Before this commit: robot cyberdog2_description, 35 links, 34 joints
Links:
- removed link FL_calf_rotor
- removed link FL_hip_rotor
- removed link FL_thigh_rotor
- removed link FL_thigh_shoulder
- removed link FR_calf_rotor
- removed link FR_hip_rotor
- removed link FR_thigh_rotor
- removed link FR_thigh_shoulder
- removed link RL_calf_rotor
- removed link RL_hip_rotor
- removed link RL_thigh_rotor
- removed link RL_thigh_shoulder
- removed link RR_calf_rotor
- removed link RR_hip_rotor
- removed link RR_thigh_rotor
- removed link RR_thigh_shoulder
- link FL_calf: geometry collision box size=0.016 0.016 0.18341; visual mesh filename=../meshes/knee.dae scale=1 1 1
- link FR_calf: geometry collision box size=0.016 0.016 0.18341; visual mesh filename=../meshes/knee.dae scale=1 1 1
- link RL_calf: geometry collision box size=0.016 0.016 0.18341; visual mesh filename=../meshes/knee.dae scale=1 1 1
- link RR_calf: geometry collision box size=0.016 0.016 0.18341; visual mesh filename=../meshes/knee.dae scale=1 1 1
Joints:
- removed joint FL_calf_rotor_fix
- removed joint FL_hip_fixed
- removed joint FL_hip_rotor_fix
- removed joint FL_thigh_rotor_fix
- removed joint FR_calf_rotor_fix
- removed joint FR_hip_fixed
- removed joint FR_hip_rotor_fix
- removed joint FR_thigh_rotor_fix
- removed joint RL_calf_rotor_fix
- removed joint RL_hip_fixed
- removed joint RL_hip_rotor_fix
- removed joint RL_thigh_rotor_fix
- removed joint RR_calf_rotor_fix
- removed joint RR_hip_fixed
- removed joint RR_hip_rotor_fix
- removed joint RR_thigh_rotor_fix

File: resources/robots/cyberdog2/xacro/const.xacro (robot description, xacro)
@@ -47,10 +47,16 @@
     <xacro:property name="hip_motorVelMax" value="30.9971" />
     <xacro:property name="knee_motorVelMax" value="30.9971" />
-    <xacro:property name="abad_damping" value="0.01" />
+    <!-- <xacro:property name="abad_damping" value="0.01" />
     <xacro:property name="hip_damping" value="0.01" />
     <xacro:property name="knee_damping" value="0.01" />
     <xacro:property name="abad_friction" value="0.1" />
     <xacro:property name="hip_friction" value="0.1" />
-    <xacro:property name="knee_friction" value="0.1" />
+    <xacro:property name="knee_friction" value="0.1" /> -->
+    <xacro:property name="abad_damping" value="0" />
+    <xacro:property name="hip_damping" value="0" />
+    <xacro:property name="knee_damping" value="0" />
+    <xacro:property name="abad_friction" value="0" />
+    <xacro:property name="hip_friction" value="0" />
+    <xacro:property name="knee_friction" value="0" />
     <!-- inertial&mass value -->
     <!-- body -->

File: resources/robots/cyberdog2/xacro/leg.xacro (robot description, xacro)
@@ -54,11 +54,11 @@
             </inertial>
         </link>
-        <joint name="${name}_hip_rotor_fix" type="fixed">
+        <!-- <joint name="${name}_hip_rotor_fix" type="fixed">
             <origin rpy="0 0 0" xyz="${-abad_rotor_offset*front_hind} 0 0" />
             <parent link="${name}_hip" />
             <child link="${name}_hip_rotor" />
-        </joint>
+        </joint> -->
         <!-- this link is only for abad rotor inertial -->
-        <link name="${name}_hip_rotor">
+        <!-- <link name="${name}_hip_rotor">
             <inertial>
                 <origin rpy="0 0 0" xyz="${rotor_com_x} ${rotor_com_y} ${rotor_com_z}" />
@@ -66,11 +66,11 @@
                 <inertia ixx="${rotor_ixx}" ixy="${rotor_ixy}" ixz="${rotor_ixz}" iyy="${rotor_iyy}" iyz="${rotor_iyz}" izz="${rotor_izz}" />
             </inertial>
-        </link>
-        <joint name="${name}_hip_fixed" type="fixed">
+        </link> -->
+        <!-- <joint name="${name}_hip_fixed" type="fixed">
             <origin rpy="0 0 0" xyz="0 ${(hip_offset-hip_shoulder_length)*mirror} 0" />
             <parent link="${name}_hip" />
             <child link="${name}_thigh_shoulder" />
-        </joint>
-        <link name="${name}_thigh_shoulder">
+        </joint> -->
+        <!-- <link name="${name}_thigh_shoulder">
             <collision>
                 <origin rpy="${PI/2.0} 0 0" xyz="0 0 0" />
@@ -79,5 +79,5 @@
                 </geometry>
             </collision>
-        </link>
+        </link> -->
         <joint name="${name}_thigh_joint" type="revolute">
             <origin rpy="0 0 0" xyz="0 ${hip_offset*mirror} 0" />
@@ -125,11 +125,11 @@
             </inertial>
         </link>
-                <joint name="${name}_thigh_rotor_fix" type="fixed">
+        <!-- <joint name="${name}_thigh_rotor_fix" type="fixed">
             <origin rpy="0 0 0" xyz="0 ${hip_rotor_offset*mirror} 0" />
             <parent link="${name}_thigh" />
             <child link="${name}_thigh_rotor" />
-        </joint>
+        </joint> -->
         <!-- this link is only for hip rotor inertial -->
-        <link name="${name}_thigh_rotor">
+        <!-- <link name="${name}_thigh_rotor">
             <inertial>
                 <origin rpy="0 0 0" xyz="${rotor_com_x} ${rotor_com_y} ${rotor_com_z}" />
@@ -137,12 +137,12 @@
                 <inertia ixx="${rotor_ixx}" ixy="${rotor_ixy}" ixz="${rotor_ixz}" iyy="${rotor_iyy}" iyz="${rotor_iyz}" izz="${rotor_izz}" />
             </inertial>
-        </link>
-        <joint name="${name}_calf_rotor_fix" type="fixed">
+        </link> -->
+        <!-- <joint name="${name}_calf_rotor_fix" type="fixed">
             <origin rpy="0 0 0" xyz="0 ${knee_rotor_offset*mirror} 0" />
             <parent link="${name}_thigh" />
             <child link="${name}_calf_rotor" />
-        </joint>
+        </joint> -->
         <!-- this link is only for knee rotor inertial -->
-        <link name="${name}_calf_rotor">
+        <!-- <link name="${name}_calf_rotor">
             <inertial>
                 <origin rpy="0 0 0" xyz="${rotor_com_x} ${rotor_com_y} ${rotor_com_z}" />
@@ -150,5 +150,5 @@
                 <inertia ixx="${rotor_ixx}" ixy="${rotor_ixy}" ixz="${rotor_ixz}" iyy="${rotor_iyy}" iyz="${rotor_iyz}" izz="${rotor_izz}" />
             </inertial>
-        </link>
+        </link> -->
         <joint name="${name}_calf_joint" type="revolute">
             <origin rpy="0 0 0" xyz="0 0 ${-hip_length}" />
@@ -175,5 +175,5 @@
                 </geometry>
             </collision>
-            <collision name="${name}_calf_rubber">
+            <!-- <collision name="${name}_calf_rubber">
                 <origin rpy="0 ${PI} 0" xyz="${-knee_rubber/2.0} 0 -0.007" />
                 <geometry>
@@ -188,5 +188,5 @@
                     </contact>
                 </surface>
-            </collision>
+            </collision> -->
             <inertial>
                 <origin rpy="0 0 0" xyz="${knee_com_x} ${knee_com_y} ${knee_com_z}" />
@@ -196,5 +196,5 @@
             </inertial>
         </link>
-        <joint name="${name}_foot_fixed" type="fixed">
+        <joint name="${name}_foot_fixed" type="fixed" dont_collapse="true">
             <origin rpy="0 0 0" xyz="0.0055 0 ${-knee_length+foot_radius/2.0}" />
             <parent link="${name}_calf" />

File: resources/robots/cyberdog2/xacro/robot.xacro (robot description, xacro)
@@ -6,4 +6,31 @@
     <xacro:include filename="leg.xacro" />
     <!-- <xacro:include filename="gazebo.xacro" /> -->
+    <material name="black">
+        <color rgba="0.0 0.0 0.0 1.0"/>
+    </material>
+    <material name="blue">
+        <color rgba="0.0 0.0 0.8 1.0"/>
+    </material>
+    <material name="green">
+        <color rgba="0.0 0.8 0.0 1.0"/>
+    </material>
+    <material name="grey">
+        <color rgba="0.2 0.2 0.2 1.0"/>
+    </material>
+    <material name="silver">
+        <color rgba="0.913725490196 0.913725490196 0.847058823529 1.0"/>
+    </material>
+    <material name="orange">
+        <color rgba="0.12 0.15 0.2 1.0"/>
+    </material>
+    <material name="brown">
+        <color rgba="0.870588235294 0.811764705882 0.764705882353 1.0"/>
+    </material>
+    <material name="red">
+        <color rgba="0.8 0.0 0.0 1.0"/>
+    </material>
+    <material name="white">
+        <color rgba="1.0 1.0 1.0 1.0"/>
+    </material>
     <link name="base">
         <visual>

Commit message: 202309082250

File: resources/robots/cyberdog2/urdf/cyberdog2.urdf (robot description, URDF)
Before this commit: robot cyberdog2_description, 35 links, 34 joints
Links:
- removed link FL_calf_rotor
- removed link FL_hip_rotor
- removed link FL_thigh_rotor
- removed link FR_calf_rotor
- removed link FR_hip_rotor
- removed link FR_thigh_rotor
- removed link RL_calf_rotor
- removed link RL_hip_rotor
- removed link RL_thigh_rotor
- removed link RR_calf_rotor
- removed link RR_hip_rotor
- removed link RR_thigh_rotor
- link FL_calf: geometry collision box size=0.016 0.016 0.18341; visual mesh filename=../meshes/knee.dae scale=1 1 1
- link FR_calf: geometry collision box size=0.016 0.016 0.18341; visual mesh filename=../meshes/knee.dae scale=1 1 1
- link RL_calf: geometry collision box size=0.016 0.016 0.18341; visual mesh filename=../meshes/knee.dae scale=1 1 1
- link RR_calf: geometry collision box size=0.016 0.016 0.18341; visual mesh filename=../meshes/knee.dae scale=1 1 1
Joints:
- removed joint FL_calf_rotor_fix
- removed joint FL_hip_rotor_fix
- removed joint FL_thigh_rotor_fix
- removed joint FR_calf_rotor_fix
- removed joint FR_hip_rotor_fix
- removed joint FR_thigh_rotor_fix
- removed joint RL_calf_rotor_fix
- removed joint RL_hip_rotor_fix
- removed joint RL_thigh_rotor_fix
- removed joint RR_calf_rotor_fix
- removed joint RR_hip_rotor_fix
- removed joint RR_thigh_rotor_fix

File: resources/robots/cyberdog2/xacro/const.xacro (robot description, xacro)
@@ -47,10 +47,16 @@
     <xacro:property name="hip_motorVelMax" value="30.9971" />
     <xacro:property name="knee_motorVelMax" value="30.9971" />
-    <xacro:property name="abad_damping" value="0.01" />
+    <xacro:property name="abad_damping" value="0.0" />
+    <xacro:property name="hip_damping" value="0.0" />
+    <xacro:property name="knee_damping" value="0.0" />
+    <xacro:property name="abad_friction" value="0.0" />
+    <xacro:property name="hip_friction" value="0.0" />
+    <xacro:property name="knee_friction" value="0.0" />
+    <!-- <xacro:property name="abad_damping" value="0.01" />
     <xacro:property name="hip_damping" value="0.01" />
     <xacro:property name="knee_damping" value="0.01" />
     <xacro:property name="abad_friction" value="0.1" />
     <xacro:property name="hip_friction" value="0.1" />
-    <xacro:property name="knee_friction" value="0.1" />
+    <xacro:property name="knee_friction" value="0.1" /> -->
     <!-- inertial&mass value -->
     <!-- body -->

File: resources/robots/cyberdog2/xacro/leg.xacro (robot description, xacro)
@@ -54,11 +54,11 @@
             </inertial>
         </link>
-        <joint name="${name}_hip_rotor_fix" type="fixed">
+        <!-- <joint name="${name}_hip_rotor_fix" type="fixed">
             <origin rpy="0 0 0" xyz="${-abad_rotor_offset*front_hind} 0 0" />
             <parent link="${name}_hip" />
             <child link="${name}_hip_rotor" />
-        </joint>
+        </joint> -->
         <!-- this link is only for abad rotor inertial -->
-        <link name="${name}_hip_rotor">
+        <!-- <link name="${name}_hip_rotor">
             <inertial>
                 <origin rpy="0 0 0" xyz="${rotor_com_x} ${rotor_com_y} ${rotor_com_z}" />
@@ -66,5 +66,5 @@
                 <inertia ixx="${rotor_ixx}" ixy="${rotor_ixy}" ixz="${rotor_ixz}" iyy="${rotor_iyy}" iyz="${rotor_iyz}" izz="${rotor_izz}" />
             </inertial>
-        </link>
+        </link> -->
         <joint name="${name}_hip_fixed" type="fixed">
             <origin rpy="0 0 0" xyz="0 ${(hip_offset-hip_shoulder_length)*mirror} 0" />
@@ -125,11 +125,11 @@
             </inertial>
         </link>
-                <joint name="${name}_thigh_rotor_fix" type="fixed">
+        <!-- <joint name="${name}_thigh_rotor_fix" type="fixed">
             <origin rpy="0 0 0" xyz="0 ${hip_rotor_offset*mirror} 0" />
             <parent link="${name}_thigh" />
             <child link="${name}_thigh_rotor" />
-        </joint>
+        </joint> -->
         <!-- this link is only for hip rotor inertial -->
-        <link name="${name}_thigh_rotor">
+        <!-- <link name="${name}_thigh_rotor">
             <inertial>
                 <origin rpy="0 0 0" xyz="${rotor_com_x} ${rotor_com_y} ${rotor_com_z}" />
@@ -137,12 +137,12 @@
                 <inertia ixx="${rotor_ixx}" ixy="${rotor_ixy}" ixz="${rotor_ixz}" iyy="${rotor_iyy}" iyz="${rotor_iyz}" izz="${rotor_izz}" />
             </inertial>
-        </link>
-        <joint name="${name}_calf_rotor_fix" type="fixed">
+        </link> -->
+        <!-- <joint name="${name}_calf_rotor_fix" type="fixed">
             <origin rpy="0 0 0" xyz="0 ${knee_rotor_offset*mirror} 0" />
             <parent link="${name}_thigh" />
             <child link="${name}_calf_rotor" />
-        </joint>
+        </joint> -->
         <!-- this link is only for knee rotor inertial -->
-        <link name="${name}_calf_rotor">
+        <!-- <link name="${name}_calf_rotor">
             <inertial>
                 <origin rpy="0 0 0" xyz="${rotor_com_x} ${rotor_com_y} ${rotor_com_z}" />
@@ -150,5 +150,5 @@
                 <inertia ixx="${rotor_ixx}" ixy="${rotor_ixy}" ixz="${rotor_ixz}" iyy="${rotor_iyy}" iyz="${rotor_iyz}" izz="${rotor_izz}" />
             </inertial>
-        </link>
+        </link> -->
         <joint name="${name}_calf_joint" type="revolute">
             <origin rpy="0 0 0" xyz="0 0 ${-hip_length}" />
@@ -175,5 +175,5 @@
                 </geometry>
             </collision>
-            <collision name="${name}_calf_rubber">
+            <!-- <collision name="${name}_calf_rubber">
                 <origin rpy="0 ${PI} 0" xyz="${-knee_rubber/2.0} 0 -0.007" />
                 <geometry>
@@ -188,5 +188,5 @@
                     </contact>
                 </surface>
-            </collision>
+            </collision> -->
             <inertial>
                 <origin rpy="0 0 0" xyz="${knee_com_x} ${knee_com_y} ${knee_com_z}" />
@@ -196,5 +196,5 @@
             </inertial>
         </link>
-        <joint name="${name}_foot_fixed" type="fixed">
+        <joint name="${name}_foot_fixed" type="fixed" dont_collapse="true">
             <origin rpy="0 0 0" xyz="0.0055 0 ${-knee_length+foot_radius/2.0}" />
             <parent link="${name}_calf" />

File: resources/robots/cyberdog2/xacro/robot.xacro (robot description, xacro)
@@ -6,4 +6,31 @@
     <xacro:include filename="leg.xacro" />
     <!-- <xacro:include filename="gazebo.xacro" /> -->
+    <material name="black">
+        <color rgba="0.0 0.0 0.0 1.0"/>
+    </material>
+    <material name="blue">
+        <color rgba="0.0 0.0 0.8 1.0"/>
+    </material>
+    <material name="green">
+        <color rgba="0.0 0.8 0.0 1.0"/>
+    </material>
+    <material name="grey">
+        <color rgba="0.2 0.2 0.2 1.0"/>
+    </material>
+    <material name="silver">
+        <color rgba="0.9137254901960784 0.9137254901960784 0.8470588235294118 1.0"/>
+    </material>
+    <material name="orange">
+        <color rgba="1.0 0.4235294117647059 0.0392156862745098 1.0"/>
+    </material>
+    <material name="brown">
+        <color rgba="0.8705882352941177 0.8117647058823529 0.7647058823529411 1.0"/>
+    </material>
+    <material name="red">
+        <color rgba="0.8 0.0 0.0 1.0"/>
+    </material>
+    <material name="white">
+        <color rgba="1.0 1.0 1.0 1.0"/>
+    </material>
     <link name="base">
         <visual>

File: resources/robots/cyberdog2/xacro/transmission.xacro (robot description, xacro)
@@ -9,5 +9,5 @@
             <actuator name="${name}_abad_motor">
             <hardwareInterface>hardware_interface/EffortJointInterface</hardwareInterface>
-            <mechanicalReduction>"${abadGearRatio}"</mechanicalReduction>
+            <mechanicalReduction>${abadGearRatio}</mechanicalReduction>
             </actuator>
         </transmission>
@@ -19,5 +19,5 @@
             <actuator name="${name}_hip_motor">
             <hardwareInterface>hardware_interface/EffortJointInterface</hardwareInterface>
-            <mechanicalReduction>"${abadGearRatio}"</mechanicalReduction>
+            <mechanicalReduction>${abadGearRatio}</mechanicalReduction>
             </actuator>
         </transmission>
@@ -29,5 +29,5 @@
             <actuator name="${name}_knee_motor">
             <hardwareInterface>hardware_interface/EffortJointInterface</hardwareInterface>
-            <mechanicalReduction>"${kneeGearRatio}"</mechanicalReduction>
+            <mechanicalReduction>${kneeGearRatio}</mechanicalReduction>
             </actuator>
         </transmission>

Commit message: feat: fuck

File: resources/robots/cyberdog2/urdf/cyberdog2.urdf (robot description, URDF)
Before this commit: robot cyberdog2_description, 23 links, 22 joints
Links:
- added link imu_link, mass 0.001; collision box size=.001 .001 .001; visual box size=0.001 0.001 0.001
Joints:
- added joint imu_joint: type fixed, parent trunk, child imu_link, origin xyz=33.4e-3 -17.2765e-3 51.0469e-3 rpy=0 0 0

File: resources/robots/cyberdog2/xacro/robot.xacro (robot description, xacro)
@@ -65,6 +65,6 @@
         </inertial>
     </link>
-    <!-- <joint name="imu_joint" type="fixed">
-        <parent link="body" />
+    <joint name="imu_joint" type="fixed">
+        <parent link="trunk" />
         <child link="imu_link" />
         <origin rpy="0 0 0" xyz="33.4e-3 -17.2765e-3 51.0469e-3" />
@@ -89,6 +89,6 @@
         </collision>
     </link>
-    <joint name="scan_joint" type="fixed">
-        <parent link="body" />
+    <!-- <joint name="scan_joint" type="fixed">
+        <parent link="trunk" />
         <child link="lidar_link" />
         <origin rpy="0 0 0" xyz="0.21425 0 0.0908" />
@@ -102,5 +102,5 @@
     </link>
     <joint name="D435_camera_joint" type="fixed">
-        <parent link="body" />
+        <parent link="trunk" />
         <child link="D435_camera_link" />
         <origin rpy="0 0 0" xyz="271.994e-3 25e-3 114.912e-3" />
@@ -126,5 +126,5 @@
     </link>
     <joint name="RGB_camera_joint" type="fixed">
-        <parent link="body" />
+        <parent link="trunk" />
         <child link="RGB_camera_link" />
         <origin rpy="0 0 0" xyz="275.76e-3 0 125.794e-3" />
@@ -150,5 +150,5 @@
     </link>
     <joint name="AI_camera_joint" type="fixed">
-        <parent link="body" />
+        <parent link="trunk" />
         <child link="AI_camera_link" />
         <origin rpy="0 0 0" xyz="290.228e-3 0 147.420e-3" />
